File: autophon-nerdblatt.kicad_pcb (KiCad board)
At the start: 2 copper layers, 265 x 140 mm, 1 part, among them J1 board-edge-connector

Commit message: schaltplan aufgeteilt, hallsensorboard erstellt, getestete logic in FF.sch erstellt.
Parts:
- added C1: C, Capacitor_SMD:C_0603_1608Metric, F.Cu at (264.0, 120.5)
- added C2: C, Capacitor_SMD:C_0603_1608Metric, F.Cu at (278.8, 120.5)
- added C3: C, Capacitor_SMD:C_0603_1608Metric, F.Cu at (293.5, 120.5)
- added C4: C, Capacitor_SMD:C_0603_1608Metric, F.Cu at (278.8, 137.2)
- added R1: R, Resistor_SMD:R_0603_1608Metric, F.Cu at (252.8, 126.3)
- added R2: R, Resistor_SMD:R_0603_1608Metric, F.Cu at (264.0, 126.0)
- added R3: R, Resistor_SMD:R_0603_1608Metric, F.Cu at (267.5, 126.5)
- added R4: R, Resistor_SMD:R_0603_1608Metric, F.Cu at (278.8, 126.0)
- added R5: R, Resistor_SMD:R_0603_1608Metric, F.Cu at (282.2, 126.5)
- added R6: R, Resistor_SMD:R_0603_1608Metric, F.Cu at (293.5, 126.0)
- added U1: 74HC74, Package_SO:SO-14_5.3x10.2mm_P1.27mm, F.Cu at (258.5, 125.2)
- added U2: L298HN, Package_TO_SOT_THT:TO-220F-15_P2.54x5.08mm_StaggerOdd_Lead5.08mm_Vertical, F.Cu at (258.5, 92.5)
- added U3: L298HN, Package_TO_SOT_THT:TO-220F-15_P2.54x5.08mm_StaggerOdd_Lead5.08mm_Vertical, F.Cu at (270.5, 92.5)
- added U4: L298HN, Package_TO_SOT_THT:TO-220F-15_P2.54x5.08mm_StaggerOdd_Lead5.08mm_Vertical, F.Cu at (282.5, 92.5)
- added U5: 74AHC04, Package_SO:SO-14_5.3x10.2mm_P1.27mm, F.Cu at (273.2, 142.0)
- added U6: 74HC74, Package_SO:SO-14_5.3x10.2mm_P1.27mm, F.Cu at (288.0, 125.2)
- added U7: 74HC74, Package_SO:SO-14_5.3x10.2mm_P1.27mm, F.Cu at (273.2, 125.2)
Routing:
- net D.1: track 0.00 -> 44.5 mm
- net Net-(U5-Pad8): track 0.00 -> 41.2 mm
- net Net-(U1-Pad2): track 0.00 -> 36.4 mm
- net D.2: track 0.00 -> 36.1 mm
- net E_IN1: track 0.00 -> 34.2 mm
- net B.1: track 0.00 -> 34.1 mm
- net B.2: track 0.00 -> 34.0 mm
- net F.2: track 0.00 -> 33.9 mm
- net C_IN1: track 0.00 -> 33.1 mm, vias 0 -> 2
- net F.1: track 0.00 -> 33.0 mm
- net Net-(U5-Pad6): track 0.00 -> 32.9 mm
- net E_IN2: track 0.00 -> 32.8 mm
- net C_IN2: track 0.00 -> 32.5 mm, vias 0 -> 2
- net A_IN1: track 0.00 -> 31.6 mm
- net A_IN2: track 0.00 -> 29.7 mm
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Other:
- net class Motor added: clearance 0.2, trace_width 1, via_dia 0.8, via_drill 0.4

Commit message: first Routing of FF
Parts:
- moved U5 5.23 mm to (273.2, 136.8)
- moved C4 5.06 mm to (278.9, 132.2)
Connections:
- U2 pad 8: GND1 -> GND
- U3 pad 8: GND1 -> GND
- U4 pad 8: GND1 -> GND
Routing:
- net +5V: track 8.40 -> 59.0 mm, vias 0 -> 4
- net D_IN3: track 0.00 -> 40.7 mm
- net D_IN4: track 0.00 -> 39.0 mm
- net Net-(U5-Pad8): track 41.2 -> 57.8 mm
- net Net-(U1-Pad12): track 24.5 -> 19.0 mm
- net Net-(U5-Pad12): track 19.7 -> 14.7 mm
- net Net-(U5-Pad10): track 24.6 -> 20.7 mm
- net Net-(U1-Pad2): track 36.4 -> 38.6 mm
- net B_IN3: track 28.8 -> 26.8 mm
- net GND: track 11.4 -> 9.44 mm, vias 0 -> 1
- net F_IN3: track 28.4 -> 26.5 mm
- net F_IN4: track 26.7 -> 25.2 mm
- net B_IN4: track 25.6 -> 24.9 mm
- net Net-(R3-Pad1): track 3.75 -> 3.08 mm
- net E_IN1: track 34.2 -> 33.6 mm
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- added copper zone on B.Cu, net GND
- added copper zone on F.Cu, net GND
Other:
- net class Default: clearance 0.2 -> 0.15; trace_width 0.25 -> 0.15; via_dia 0.8 -> 0.3; via_drill 0.4 -> 0.2
- rule trace_clearance: 0.2 -> 0.15
- rule trace_min: 0.2 -> 0.15
- rule via_min_drill: 0.3 -> 0.2
- rule via_min_size: 0.4 -> 0.3
