File: dummy_vogelchr.sch (KiCad schematic (older format))
At the start: 14 parts

Commit message: Minor cleanup, adding the w1_test_pcb_lib, just for the single gate buffer.
Parts:
- removed U? (x2): 74LS07, symbol 74xx:74LS07
- added C?: C, symbol Device:C
- added D? (x2): 5v1, symbol Device:D_Zener
- added R?: 10k, symbol Device:R
- added U? (x3): SN74LV1T34, Package_TO_SOT_SMD:SOT-23-5, symbol w1_test_pcb_lib:SN74LV1T34
- added U?: AZ1117-3.3, symbol Regulator_Linear:AZ1117-3.3
- R?: value 10k -> 51R
- R?: value R -> 10k
Connections:
- wire segments 108 -> 127
Other:
- note added: "This circuit 3 times"
- note added: "WARNING:\nThose are just placeholders, choose the correct MCU ports!"
- note added: "be sure to use T type family!"
- moved on the sheet: R?, U?
